Commit message: added new configuration folder

File: utils/alterego_moveit_config/config/gazebo_ego_robot.urdf (robot description, URDF)
Before this commit: robot ego_robot, 123 links, 122 joints
Links:
- link back_kick_stand: geometry collision mesh filename=package://alterego_description/meshes/alterego_v3/collision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 scale=0.001 0.001 0.001; visual mesh filename=package://alterego_description/meshes/alterego_v3/visual/sa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 scale=0.001 0.001 0.001
- link back_wheel: geometry collision mesh filename=package://alterego_description/meshes/alterego_v3/collision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 scale=0.001 0.001 0.001; visual mesh filename=package://alterego_description/meshes/alterego_v3/visual/gy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 scale=0.001 0.001 0.001
- link base_link: geometry collision mesh filename=package://alterego_description/meshes/alterego_v3/collision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 scale=0.001 0.001 0.001; visual mesh filename=package://alterego_description/meshes/alterego_v3/visual/ae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 scale=0.001 0.001 0.001
- link camera_link: geometry collision box size=0.02505 0.09 0.025; visual mesh filename=package://alterego_description/meshes/common/visual/d415.stl
- link front_kick_stand: geometry collision mesh filename=package://alterego_description/meshes/alterego_v3/collision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 scale=0.001 0.001 0.001; visual mesh filename=package://alterego_description/meshes/alterego_v3/visual/sa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 scale=0.001 0.001 0.001
- link front_wheel: geometry collision mesh filename=package://alterego_description/meshes/alterego_v3/collision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 scale=0.001 0.001 0.001; visual mesh filename=package://alterego_description/meshes/alterego_v3/visual/gy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 scale=0.001 0.001 0.001
- link head_robot: geometry collision mesh filename=package://alterego_description/meshes/alterego_v3/collision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 scale=0.001 0.001 0.001; visual mesh filename=package://alterego_description/meshes/alterego_v3/visual/mt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 scale=0.001 0.001 0.001
- link imu: geometry collision mesh filename=package://alterego_description/meshes/common/collision/mc_s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 scale=0.001 0.001 0.001; visual mesh filename=package://alterego_description/meshes/common/visual/mc_seg_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 scale=0.001 0.001 0.001
- link left_arm_cube: geometry collision box size=0.07 0.07 0.07; visual mesh filename=package://alterego_description/meshes/common/visual/qb_move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 scale=0.001 0.001 0.001
- link left_arm_flange: geometry collision mesh filename=package://alterego_description/meshes/alterego_v3/collision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 scale=0.001 0.001 0.001; visual mesh filename=package://alterego_description/meshes/alterego_v3/visual/la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 scale=0.001 0.001 0.001
- link left_elbow_cube: geometry collision box size=0.07 0.07 0.07; visual mesh filename=package://alterego_description/meshes/common/visual/qb_move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 scale=0.001 0.001 0.001
- link left_elbow_flange: geometry collision mesh filename=package://alterego_description/meshes/common/collision/la_f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 scale=0.001 0.001 0.001; visual mesh filename=package://alterego_description/meshes/common/visual/la_flg_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 scale=0.001 0.001 0.001
- link left_elbow_flange_sensor: geometry collision mesh filename=package://alterego_description/meshes/alterego_v3/collision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 scale=0.001 0.001 0.001; visual mesh filename=package://alterego_description/meshes/alterego_v3/visual/fs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 scale=0.001 0.001 0.001
- link left_forearm_cube: geometry collision box size=0.07 0.07 0.07; visual mesh filename=package://alterego_description/meshes/common/visual/qb_move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 scale=0.001 0.001 0.001
- link left_forearm_flange: geometry collision mesh filename=package://alterego_description/meshes/common/collision/la_f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 scale=0.001 0.001 0.001; visual mesh filename=package://alterego_description/meshes/common/visual/la_flg_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 scale=0.001 0.001 0.001
- link left_shoulder_cube: geometry collision box size=0.07 0.07 0.07; visual mesh filename=package://alterego_description/meshes/alterego_v3/visual/qb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 scale=0.001 0.001 0.001
- link left_shoulder_flange: geometry collision mesh filename=package://alterego_description/meshes/common/collision/la_f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 scale=0.001 0.001 0.001; visual mesh filename=package://alterego_description/meshes/common/visual/la_flg_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 scale=0.001 0.001 0.001
- link left_wrist: geometry collision mesh filename=package://alterego_description/meshes/alterego_v3/collision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 scale=0.001 0.001 0.001; visual mesh filename=package://alterego_description/meshes/alterego_v3/visual/le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 scale=0.001 0.001 0.001
- link left_wrist_flange: geometry collision mesh filename=package://alterego_description/meshes/common/collision/la_f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 scale=0.001 0.001 0.001; visual mesh filename=package://alterego_description/meshes/common/visual/la_flg_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 scale=0.001 0.001 0.001
- link neck: geometry collision mesh filename=package://alterego_description/meshes/alterego_v3/collision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 scale=0.001 0.001 0.001; visual mesh filename=package://alterego_description/meshes/alterego_v3/visual/fl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 scale=0.001 0.001 0.001
- link neck_cube: geometry collision box size=0.07 0.07 0.07; visual mesh filename=package://alterego_description/meshes/common/visual/qb_move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 scale=0.001 0.001 0.001
- link right_arm_cube: geometry collision box size=0.07 0.07 0.07; visual mesh filename=package://alterego_description/meshes/common/visual/qb_move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 scale=0.001 0.001 0.001
- link right_arm_flange: geometry collision mesh filename=package://alterego_description/meshes/alterego_v3/collision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 scale=0.001 0.001 0.001; visual mesh filename=package://alterego_description/meshes/alterego_v3/visual/la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 scale=0.001 0.001 0.001
- link right_elbow_cube: geometry collision box size=0.07 0.07 0.07; visual mesh filename=package://alterego_description/meshes/common/visual/qb_move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 scale=0.001 0.001 0.001
- link right_elbow_flange: geometry collision mesh filename=package://alterego_description/meshes/common/collision/la_f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 scale=0.001 0.001 0.001; visual mesh filename=package://alterego_description/meshes/common/visual/la_flg_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 scale=0.001 0.001 0.001
- link right_elbow_flange_sensor: geometry collision mesh filename=package://alterego_description/meshes/alterego_v3/collision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 scale=0.001 0.001 0.001; visual mesh filename=package://alterego_description/meshes/alterego_v3/visual/fs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 scale=0.001 0.001 0.001
- link right_forearm_cube: geometry collision box size=0.07 0.07 0.07; visual mesh filename=package://alterego_description/meshes/common/visual/qb_move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 scale=0.001 0.001 0.001
- link right_forearm_flange: geometry collision mesh filename=package://alterego_description/meshes/common/collision/la_f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 scale=0.001 0.001 0.001; visual mesh filename=package://alterego_description/meshes/common/visual/la_flg_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 scale=0.001 0.001 0.001
- link right_shoulder_cube: geometry collision box size=0.07 0.07 0.07; visual mesh filename=package://alterego_description/meshes/alterego_v3/visual/qb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 scale=0.001 0.001 0.001
- link right_shoulder_flange: geometry collision mesh filename=package://alterego_description/meshes/common/collision/la_f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 scale=0.001 0.001 0.001; visual mesh filename=package://alterego_description/meshes/common/visual/la_flg_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 scale=0.001 0.001 0.001
- link right_wrist: geometry collision mesh filename=package://alterego_description/meshes/alterego_v3/collision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 scale=0.001 0.001 0.001; visual mesh filename=package://alterego_description/meshes/alterego_v3/visual/ri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 scale=0.001 0.001 0.001
- link right_wrist_flange: geometry collision mesh filename=package://alterego_description/meshes/common/collision/la_f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 scale=0.001 0.001 0.001; visual mesh filename=package://alterego_description/meshes/common/visual/la_flg_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 scale=0.001 0.001 0.001
- link scan: geometry collision mesh filename=package://alterego_description/meshes/common/collision/rpli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 scale=0.001 0.001 0.001; visual mesh filename=package://alterego_description/meshes/common/visual/rplidar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 scale=0.001 0.001 0.001
- link wheel_L: geometry collision cylinder length=0.07 radius=0.13; visual mesh filename=package://alterego_description/meshes/common/visual/mteg100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 scale=0.001 0.001 0.001
- link wheel_R: geometry collision cylinder length=0.07 radius=0.13; visual mesh filename=package://alterego_description/meshes/common/visual/mteg100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 scale=0.001 0.001 0.001
- link zed: geometry collision mesh filename=package://alterego_description/meshes/common/collision/zedm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 scale=0.001 0.001 0.001; visual mesh filename=package://alterego_description/meshes/common/visual/zedm.dae scale=0.001 0.001 0.001

File: utils/ego_dance/urdf/ego_robot_gazebo_v2.urdf (robot description, URDF)
Before this commit: robot alterego, 44 links, 43 joints
Links:
- link base: geometry collision mesh filename=package://alterego_description/meshes/alterego_v2/collision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 scale=0.001 0.001 0.001; visual mesh filename=package://alterego_description/meshes/alterego_v2/visual/bo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 scale=0.001 0.001 0.001
- link camera: geometry collision mesh filename=package://alterego_description/meshes/common/collision/zedm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 scale=0.001 0.001 0.001; visual mesh filename=package://alterego_description/meshes/common/visual/zedm.dae scale=0.001 0.001 0.001
- link head: geometry collision mesh filename=package://alterego_description/meshes/alterego_v2/collision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 scale=0.001 0.001 0.001; visual mesh filename=package://alterego_description/meshes/alterego_v2/visual/mt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 scale=0.001 0.001 0.001
- link imu: geometry collision mesh filename=package://alterego_description/meshes/common/collision/mc_s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 scale=0.001 0.001 0.001; visual mesh filename=package://alterego_description/meshes/common/visual/mc_seg_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 scale=0.001 0.001 0.001
- link laser: geometry collision mesh filename=package://alterego_description/meshes/common/collision/rpli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 scale=0.001 0.001 0.001; visual mesh filename=package://alterego_description/meshes/common/visual/rplidar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 scale=0.001 0.001 0.001
- link left_arm_cube: geometry collision box size=0.07 0.07 0.07; visual mesh filename=package://alterego_description/meshes/common/visual/qb_move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 scale=0.001 0.001 0.001
- link left_arm_flange: geometry collision mesh filename=package://alterego_description/meshes/common/collision/la_f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 scale=0.001 0.001 0.001; visual mesh filename=package://alterego_description/meshes/common/visual/la_flg_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 scale=0.001 0.001 0.001
- link left_elbow_cube: geometry collision box size=0.07 0.07 0.07; visual mesh filename=package://alterego_description/meshes/common/visual/qb_move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 scale=0.001 0.001 0.001
- link left_elbow_flange: geometry collision mesh filename=package://alterego_description/meshes/common/collision/la_f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 scale=0.001 0.001 0.001; visual mesh filename=package://alterego_description/meshes/common/visual/la_flg_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 scale=0.001 0.001 0.001
- link left_forearm_cube: geometry collision box size=0.07 0.07 0.07; visual mesh filename=package://alterego_description/meshes/common/visual/qb_move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 scale=0.001 0.001 0.001
- link left_forearm_flange: geometry collision mesh filename=package://alterego_description/meshes/common/collision/la_f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 scale=0.001 0.001 0.001; visual mesh filename=package://alterego_description/meshes/common/visual/la_flg_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 scale=0.001 0.001 0.001
- link left_forearm_hand_flange: geometry collision mesh filename=package://alterego_description/meshes/alterego_v2/collision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 scale=0.001 0.001 0.001; visual mesh filename=package://alterego_description/meshes/alterego_v2/visual/mc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 scale=0.001 0.001 0.001
- link left_hand: geometry collision mesh filename=package://alterego_description/meshes/common/collision/soft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 scale=0.001 0.001 0.001; visual mesh filename=package://alterego_description/meshes/common/visual/softhan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 scale=0.001 0.001 0.001
- link left_shoulder_cube: geometry collision box size=0.07 0.07 0.07; visual mesh filename=package://alterego_description/meshes/common/visual/qb_move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 scale=0.001 0.001 0.001
- link left_shoulder_flange: geometry collision mesh filename=package://alterego_description/meshes/common/collision/la_f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 scale=0.001 0.001 0.001; visual mesh filename=package://alterego_description/meshes/common/visual/la_flg_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 scale=0.001 0.001 0.001
- link left_wrist_flange: geometry collision mesh filename=package://alterego_description/meshes/common/collision/la_f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 scale=0.001 0.001 0.001; visual mesh filename=package://alterego_description/meshes/common/visual/la_flg_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 scale=0.001 0.001 0.001
- link neck: geometry collision mesh filename=package://alterego_description/meshes/common/collision/la_f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 scale=0.001 0.001 0.001; visual mesh filename=package://alterego_description/meshes/common/visual/la_flg_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 scale=0.001 0.001 0.001
- link neck_cube: geometry collision box size=0.07 0.07 0.07; visual mesh filename=package://alterego_description/meshes/common/visual/qb_move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 scale=0.001 0.001 0.001
- link realsense: geometry collision mesh filename=package://alterego_description/meshes/common/collision/inte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 scale=0.001 0.001 0.001; visual mesh filename=package://alterego_description/meshes/common/visual/intel_r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 scale=0.001 0.001 0.001
- link right_arm_cube: geometry collision box size=0.07 0.07 0.07; visual mesh filename=package://alterego_description/meshes/common/visual/qb_move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 scale=0.001 0.001 0.001
- link right_arm_flange: geometry collision mesh filename=package://alterego_description/meshes/common/collision/la_f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 scale=0.001 0.001 0.001; visual mesh filename=package://alterego_description/meshes/common/visual/la_flg_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 scale=0.001 0.001 0.001
- link right_elbow_cube: geometry collision box size=0.07 0.07 0.07; visual mesh filename=package://alterego_description/meshes/common/visual/qb_move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 scale=0.001 0.001 0.001
- link right_elbow_flange: geometry collision mesh filename=package://alterego_description/meshes/common/collision/la_f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 scale=0.001 0.001 0.001; visual mesh filename=package://alterego_description/meshes/common/visual/la_flg_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 scale=0.001 0.001 0.001
- link right_forearm_cube: geometry collision box size=0.07 0.07 0.07; visual mesh filename=package://alterego_description/meshes/common/visual/qb_move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 scale=0.001 0.001 0.001
- link right_forearm_flange: geometry collision mesh filename=package://alterego_description/meshes/common/collision/la_f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 scale=0.001 0.001 0.001; visual mesh filename=package://alterego_description/meshes/common/visual/la_flg_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 scale=0.001 0.001 0.001
- link right_forearm_hand_flange: geometry collision mesh filename=package://alterego_description/meshes/alterego_v2/collision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 scale=0.001 0.001 0.001; visual mesh filename=package://alterego_description/meshes/alterego_v2/visual/mc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 scale=0.001 0.001 0.001
- link right_hand: geometry collision mesh filename=package://alterego_description/meshes/common/collision/soft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 scale=0.001 0.001 0.001; visual mesh filename=package://alterego_description/meshes/common/visual/softhan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 scale=0.001 0.001 0.001
- link right_shoulder_cube: geometry collision box size=0.07 0.07 0.07; visual mesh filename=package://alterego_description/meshes/common/visual/qb_move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 scale=0.001 0.001 0.001
- link right_shoulder_flange: geometry collision mesh filename=package://alterego_description/meshes/common/collision/la_f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 scale=0.001 0.001 0.001; visual mesh filename=package://alterego_description/meshes/common/visual/la_flg_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 scale=0.001 0.001 0.001
- link right_wrist_flange: geometry collision mesh filename=package://alterego_description/meshes/common/collision/la_f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 scale=0.001 0.001 0.001; visual mesh filename=package://alterego_description/meshes/common/visual/la_flg_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 scale=0.001 0.001 0.001
- link wheel_L: geometry collision cylinder length=0.07 radius=0.13; visual mesh filename=package://alterego_description/meshes/common/visual/mteg100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 scale=0.001 0.001 0.001
- link wheel_R: geometry collision cylinder length=0.07 radius=0.13; visual mesh filename=package://alterego_description/meshes/common/visual/mteg100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 scale=0.001 0.001 0.001
